File: Hardware/DualWatch/nrf5340_QKAA.kicad_sch (KiCad schematic)
At the start: 47 parts, among them J1 NFC, J1 USB_C_Receptacle_USB2.0, J3 NRF_Debug, U1 NRF5340-QKAA-R7, Y2 32MHz, Y3 32.768kHz

Commit message: update pcb
Changed lines of the file:
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@@
     (stroke (width 0) (type default))
   )
-  (wire (pts (xy 259.715 180.34) (xy 263.525 180.34))
+  (wire (pts (xy 253.365 180.34) (xy 263.525 180.34))
     (stroke (width 0) (type default))
   )
@@
     (stroke (width 0) (type default))
   )
-  (wire (pts (xy 259.715 177.8) (xy 263.525 177.8))
+  (wire (pts (xy 253.365 177.8) (xy 263.525 177.8))
     (stroke (width 0) (type default))
   )
@@
     (effects (font (size 1.27 1.27)) (justify left bottom))
   )
+  (label "USB_D+" (at 253.365 180.34 0) (fields_autoplaced)
+    (effects (font (size 1.27 1.27)) (justify left bottom))
+  )
   (label "NRESET" (at 253.365 165.1 0) (fields_autoplaced)
     (effects (font (size 1.27 1.27)) (justify left bottom))
+  )
+  (label "USB_D-" (at 267.97 252.73 180) (fields_autoplaced)
+    (effects (font (size 1.27 1.27)) (justify right bottom))
   )
   (label "XL1" (at 129.54 260.985 180) (fields_autoplaced)
@@
     (effects (font (size 1.27 1.27)) (justify left bottom))
   )
+  (label "USB_D-" (at 253.365 177.8 0) (fields_autoplaced)
+    (effects (font (size 1.27 1.27)) (justify left bottom))
+  )
   (label "XC2" (at 253.365 147.32 0) (fields_autoplaced)
     (effects (font (size 1.27 1.27)) (justify left bottom))
@@
   (label "NFC1" (at 97.79 42.545 0) (fields_autoplaced)
     (effects (font (size 1.27 1.27)) (justify left bottom))
+  )
+  (label "USB_D+" (at 267.97 257.81 180) (fields_autoplaced)
+    (effects (font (size 1.27 1.27)) (justify right bottom))
   )
   (label "SWDCLK" (at 70.485 259.715 0) (fields_autoplaced)
@@
     (effects (font (size 1.27 1.27)) (justify right))
   )
-  (hierarchical_label "USB_D-" (shape input) (at 259.715 177.8 180) (fields_autoplaced)
-    (effects (font (size 1.27 1.27)) (justify right))
-  )
   (hierarchical_label "P0.18{slash}CSN" (shape input) (at 96.52 83.185 180) (fields_autoplaced)
     (effects (font (size 1.27 1.27)) (justify right))
@@
     (effects (font (size 1.27 1.27)) (justify right))
   )
-  (hierarchical_label "USB_D+" (shape input) (at 267.97 257.81 0) (fields_autoplaced)
-    (effects (font (size 1.27 1.27)) (justify left))
-  )
   (hierarchical_label "P0.08{slash}SCK" (shape input) (at 96.52 57.785 180) (fields_autoplaced)
     (effects (font (size 1.27 1.27)) (justify right))
@@
     (effects (font (size 1.27 1.27)) (justify right))
   )
-  (hierarchical_label "USB_D+" (shape input) (at 259.715 180.34 180) (fields_autoplaced)
-    (effects (font (size 1.27 1.27)) (justify right))
-  )
   (hierarchical_label "P0.29" (shape input) (at 91.44 111.125 180) (fields_autoplaced)
     (effects (font (size 1.27 1.27)) (justify right))
@@
     (effects (font (size 1.27 1.27)) (justify right))
   )
-  (hierarchical_label "USB_D-" (shape input) (at 267.97 252.73 0) (fields_autoplaced)
-    (effects (font (size 1.27 1.27)) (justify left))
-  )
   (symbol (lib_id "Device:C") (at 144.78 182.88 0) (unit 1)
