File: Hardware/DualWatch/lis3dh.kicad_sch (KiCad schematic)
At the start: 4 parts, among them U5 LIS3DH

Commit message: Update Schematic
Parts:
- removed U5: LIS3DH, Package_LGA:LGA-16_3x3mm_P0.5mm_LayoutBorder3x5y, symbol Sensor_Motion:LIS3DH
- added U7: LIS3DH, Package_LGA:LGA-16_3x3mm_P0.5mm_LayoutBorder3x5y, symbol Sensor_Motion:LIS3DH
- renumbered C46 to C48, C47 to C49, C48 to C50
Connections:
- net +1V8: now also U7.1 (VDD_IO)
- net +3V3: now also U7.14 (VDD), U7.15 (ADC2), U7.7 (SDO/SA0), U7.8 (CS)
- net GND: now also U7.10 (GND), U7.12 (GND), U7.13 (ADC3), U7.16 (ADC1), U7.5 (GND)
- net INT1: now also U7.11 (INT1)
- net INT2: now also U7.9 (INT2)
- net SCL: now also U7.4 (SCL/SPC)
- net SDA: now also U7.6 (SDA/SDI/SDO)
Changed lines of the file:
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@@
   (symbol (lib_id "power:GND") (at 151.13 122.555 0) (unit 1)
     (in_bom yes) (on_board yes) (dnp no) (fields_autoplaced)
-    (property "Reference" "#PWR042" (at 151.13 128.905 0)
+    (property "Reference" "#PWR048" (at 151.13 128.905 0)
       (effects (font (size 1.27 1.27)) hide)
     )
@@
       (project "DualWatch"
         (path "/9c47ae17-f150-4290-a1ee-d756173e0f3d/5cd2a7de-33fe-4e4e-987a-f156d102a916"
-          (reference "#PWR042") (unit 1)
+          (reference "#PWR048") (unit 1)
         )
       )
@@
   (symbol (lib_id "Device:C") (at 160.02 86.36 90) (unit 1)
     (in_bom yes) (on_board yes) (dnp no) (fields_autoplaced)
-    (property "Reference" "C48" (at 160.02 78.74 90)
+    (property "Reference" "C50" (at 160.02 78.74 90)
       (effects (font (size 1.27 1.27)))
     )
@@
       (project "DualWatch"
         (path "/9c47ae17-f150-4290-a1ee-d756173e0f3d/5cd2a7de-33fe-4e4e-987a-f156d102a916"
-          (reference "C48") (unit 1)
+          (reference "C50") (unit 1)
         )
       )
@@
     )
   )
+  (symbol (lib_name "LIS3DH_1") (lib_id "Sensor_Motion:LIS3DH") (at 151.13 101.6 0) (unit 1)
+    (in_bom yes) (on_board yes) (dnp no) (fields_autoplaced)
+    (property "Reference" "U7" (at 153.3241 116.84 0)
+      (effects (font (size 1.27 1.27)) (justify left))
+    )
+    (property "Value" "LIS3DH" (at 153.3241 119.38 0)
+      (effects (font (size 1.27 1.27)) (justify left))
+    )
+    (property "Footprint" "Package_LGA:LGA-16_3x3mm_P0.5mm_LayoutBorder3x5y" (at 153.67 128.27 0)
+      (effects (font (size 1.27 1.27)) hide)
+    )
+    (property "Datasheet" "https://www.st.com/resource/en/datasheet/cd00274221.pdf" (at 146.05 104.14 0)
+      (effects (font (size 1.27 1.27)) hide)
+    )
+    (pin "15")
+    (pin "8")
+    (pin "12")
+    (pin "14")
+    (pin "5")
+    (pin "10")
+    (pin "7")
+    (pin "6")
+    (pin "9")
+    (pin "2")
+    (pin "4")
+    (pin "1")
+    (pin "3")
+    (pin "13")
+    (pin "11")
+    (pin "16")
+    (instances
+      (project "DualWatch"
+        (path "/9c47ae17-f150-4290-a1ee-d756173e0f3d/5cd2a7de-33fe-4e4e-987a-f156d102a916"
+          (reference "U7") (unit 1)
+        )
+      )
+    )
+  )
   (symbol (lib_id "power:+3V3") (at 153.67 70.485 0) (unit 1)
     (in_bom yes) (on_board yes) (dnp no) (fields_autoplaced)
-    (property "Reference" "#PWR041" (at 153.67 74.295 0)
+    (property "Reference" "#PWR049" (at 153.67 74.295 0)
       (effects (font (size 1.27 1.27)) hide)
     )
@@
       (project "DualWatch"
         (path "/9c47ae17-f150-4290-a1ee-d756173e0f3d/5cd2a7de-33fe-4e4e-987a-f156d102a916"
-          (reference "#PWR041") (unit 1)
+          (reference "#PWR049") (unit 1)
         )
       )
@@
   (symbol (lib_id "power:+3V3") (at 130.175 111.76 180) (unit 1)
     (in_bom yes) (on_board yes) (dnp no) (fields_autoplaced)
-    (property "Reference" "#PWR012" (at 130.175 107.95 0)
+    (property "Reference" "#PWR045" (at 130.175 107.95 0)
       (effects (font (size 1.27 1.27)) hide)
     )
@@
       (project "DualWatch"
         (path "/9c47ae17-f150-4290-a1ee-d756173e0f3d/5cd2a7de-33fe-4e4e-987a-f156d102a916"
-          (reference "#PWR012") (unit 1)
+          (reference "#PWR045") (unit 1)
         )
       )
@@
   (symbol (lib_id "power:GND") (at 170.18 88.9 0) (unit 1)
     (in_bom yes) (on_board yes) (dnp no) (fields_autoplaced)
-    (property "Reference" "#PWR044" (at 170.18 95.25 0)
+    (property "Reference" "#PWR051" (at 170.18 95.25 0)
       (effects (font (size 1.27 1.27)) hide)
     )
@@
       (project "DualWatch"
         (path "/9c47ae17-f150-4290-a1ee-d756173e0f3d/5cd2a7de-33fe-4e4e-987a-f156d102a916"
-          (reference "#PWR044") (unit 1)
-        )
-      )
-    )
-  )
-  (symbol (lib_id "Sensor_Motion:LIS3DH") (at 151.13 101.6 0) (unit 1)
-    (in_bom yes) (on_board yes) (dnp no) (fields_autoplaced)
-    (property "Reference" "U5" (at 153.1494 117.475 0)
-      (effects (font (size 1.27 1.27)) (justify left))
-    )
-    (property "Value" "LIS3DH" (at 153.1494 120.015 0)
-      (effects (font (size 1.27 1.27)) (justify left))
-    )
-    (property "Footprint" "Package_LGA:LGA-16_3x3mm_P0.5mm_LayoutBorder3x5y" (at 153.67 128.27 0)
-      (effects (font (size 1.27 1.27)) hide)
-    )
-    (property "Datasheet" "https://www.st.com/resource/en/datasheet/cd00274221.pdf" (at 146.05 104.14 0)
-      (effects (font (size 1.27 1.27)) hide)
-    )
-    (pin "1")
-    (pin "10")
-    (pin "11")
-    (pin "12")
-    (pin "13")
-    (pin "14")
-    (pin "15")
-    (pin "16")
-    (pin "2")
-    (pin "3")
-    (pin "4")
-    (pin "5")
-    (pin "6")
-    (pin "7")
-    (pin "8")
-    (pin "9")
-    (instances
-      (project "DualWatch"
-        (path "/9c47ae17-f150-4290-a1ee-d756173e0f3d/5cd2a7de-33fe-4e4e-987a-f156d102a916"
-          (reference "U5") (unit 1)
-        )
-      )
-      (project "lis3dhtr_default"
-        (path "/b2685f9a-e85c-4296-8363-23afe10ab821"
-          (reference "U1") (unit 1)
+          (reference "#PWR051") (unit 1)
         )
       )
@@
   (symbol (lib_id "power:+1V8") (at 148.59 74.93 0) (unit 1)
     (in_bom yes) (on_board yes) (dnp no) (fields_autoplaced)
-    (property "Reference" "#PWR049" (at 148.59 78.74 0)
+    (property "Reference" "#PWR047" (at 148.59 78.74 0)
       (effects (font (size 1.27 1.27)) hide)
     )
@@
       (project "DualWatch"
         (path "/9c47ae17-f150-4290-a1ee-d756173e0f3d/5cd2a7de-33fe-4e4e-987a-f156d102a916"
-          (reference "#PWR049") (unit 1)
+          (reference "#PWR047") (unit 1)
         )
       )
@@
   (symbol (lib_id "power:+3V3") (at 172.085 101.6 270) (unit 1)
     (in_bom yes) (on_board yes) (dnp no) (fields_autoplaced)
-    (property "Reference" "#PWR045" (at 168.275 101.6 0)
+    (property "Reference" "#PWR052" (at 168.275 101.6 0)
       (effects (font (size 1.27 1.27)) hide)
     )
@@
       (project "DualWatch"
         (path "/9c47ae17-f150-4290-a1ee-d756173e0f3d/5cd2a7de-33fe-4e4e-987a-f156d102a916"
-          (reference "#PWR045") (unit 1)
+          (reference "#PWR052") (unit 1)
         )
       )
@@
   (symbol (lib_id "Device:C") (at 142.875 82.55 270) (unit 1)
     (in_bom yes) (on_board yes) (dnp no) (fields_autoplaced)
-    (property "Reference" "C46" (at 142.875 74.93 90)
+    (property "Reference" "C48" (at 142.875 74.93 90)
       (effects (font (size 1.27 1.27)))
     )
@@
       (project "DualWatch"
         (path "/9c47ae17-f150-4290-a1ee-d756173e0f3d/5cd2a7de-33fe-4e4e-987a-f156d102a916"
-          (reference "C46") (unit 1)
+          (reference "C48") (unit 1)
         )
       )
@@
   (symbol (lib_id "power:GND") (at 137.16 82.55 270) (unit 1)
     (in_bom yes) (on_board yes) (dnp no) (fields_autoplaced)
-    (property "Reference" "#PWR040" (at 130.81 82.55 0)
+    (property "Reference" "#PWR046" (at 130.81 82.55 0)
       (effects (font (size 1.27 1.27)) hide)
     )
@@
       (project "DualWatch"
         (path "/9c47ae17-f150-4290-a1ee-d756173e0f3d/5cd2a7de-33fe-4e4e-987a-f156d102a916"
-          (reference "#PWR040") (unit 1)
+          (reference "#PWR046") (unit 1)
         )
       )
@@
   (symbol (lib_id "Device:C") (at 160.02 74.93 90) (unit 1)
     (in_bom yes) (on_board yes) (dnp no) (fields_autoplaced)
-    (property "Reference" "C47" (at 160.02 67.31 90)
+    (property "Reference" "C49" (at 160.02 67.31 90)
       (effects (font (size 1.27 1.27)))
     )
@@
       (project "DualWatch"
         (path "/9c47ae17-f150-4290-a1ee-d756173e0f3d/5cd2a7de-33fe-4e4e-987a-f156d102a916"
-          (reference "C47") (unit 1)
+          (reference "C49") (unit 1)
         )
       )
@@
   (symbol (lib_id "power:GND") (at 168.275 107.95 0) (unit 1)
     (in_bom yes) (on_board yes) (dnp no) (fields_autoplaced)
-    (property "Reference" "#PWR043" (at 168.275 114.3 0)
+    (property "Reference" "#PWR050" (at 168.275 114.3 0)
       (effects (font (size 1.27 1.27)) hide)
     )
@@
       (project "DualWatch"
         (path "/9c47ae17-f150-4290-a1ee-d756173e0f3d/5cd2a7de-33fe-4e4e-987a-f156d102a916"
-          (reference "#PWR043") (unit 1)
-        )
-      )
+          (reference "#PWR050") (unit 1)
+        )
+      )

Commit message: update pcb placing
Parts:
- C48, C50: footprint Capacitor_SMD:C_0603_1608Metric -> Capacitor_SMD:C_0402_1005Metric
Changed lines of the file:
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@@
       (effects (font (size 1.27 1.27)))
     )
-    (property "Footprint" "Capacitor_SMD:C_0603_1608Metric" (at 163.83 85.3948 0)
+    (property "Footprint" "Capacitor_SMD:C_0402_1005Metric" (at 163.83 85.3948 0)
       (effects (font (size 1.27 1.27)) hide)
     )
@@
       (effects (font (size 1.27 1.27)))
     )
-    (property "Footprint" "Capacitor_SMD:C_0603_1608Metric" (at 139.065 83.5152 0)
+    (property "Footprint" "Capacitor_SMD:C_0402_1005Metric" (at 139.065 83.5152 0)
       (effects (font (size 1.27 1.27)) hide)
     )
