File: Hardware/DualWatch/nrf7002-qfaa-r7.kicad_sch (KiCad schematic)
At the start: 28 parts, among them U3 74LVC1G3157, U4 NRF7002-QFAA-R, U6 DPX165950DT-8126A1, Y2 40Mhz

Commit message: Update Schematic
Parts:
- C30: renamed from C28; footprint Capacitor_SMD:C_0402_1005Metric -> Capacitor_SMD:C_0603_1608Metric
- C33: renamed from C31; footprint Capacitor_SMD:C_0402_1005Metric -> Capacitor_SMD:C_0603_1608Metric
- C34: renamed from C32; footprint Capacitor_SMD:C_0603_1608Metric -> Capacitor_SMD:C_0402_1005Metric
- C35: renamed from C33; footprint Capacitor_SMD:C_0603_1608Metric -> Capacitor_SMD:C_0402_1005Metric
- C36: renamed from C34; footprint Capacitor_SMD:C_0402_1005Metric -> Capacitor_SMD:C_0603_1608Metric
- C37: renamed from C35; footprint Capacitor_SMD:C_0402_1005Metric -> Capacitor_SMD:C_0603_1608Metric
- C43: renamed from C41; footprint Capacitor_SMD:C_0603_1608Metric -> Capacitor_SMD:C_0402_1005Metric
- C44: renamed from C42; footprint Capacitor_SMD:C_0603_1608Metric -> Capacitor_SMD:C_0402_1005Metric
- C45: renamed from C43; footprint Capacitor_SMD:C_0402_1005Metric -> Capacitor_SMD:C_0603_1608Metric
- C46: renamed from C44; footprint Capacitor_SMD:C_0402_1005Metric -> Capacitor_SMD:C_0603_1608Metric
- L5: footprint Inductor_SMD:L_0603_1608Metric -> Inductor_SMD:L_0402_1005Metric
- L6: footprint Inductor_SMD:L_0402_1005Metric -> Inductor_SMD:L_0805_2012Metric
- L9: renamed from L8; footprint Inductor_SMD:L_0805_2012Metric -> Inductor_SMD:L_0603_1608Metric
- U5: renamed from U6; footprint DPX165950DT-8126A1:DPX-6_1P6X0P8 -> Package_LGA:LGA-16_3x3mm_P0.5mm_LayoutBorder3x5y
- renumbered C27 to C29, C29 to C31, C30 to C32, C36 to C38, C37 to C39, C38 to C40, C39 to C41, C40 to C42, C45 to C47

Commit message: Update pcb
Parts:
- U5: footprint Package_LGA:LGA-16_3x3mm_P0.5mm_LayoutBorder3x5y -> DPX165950DT-8126A1:DPX-6_1P6X0P8
Changed lines of the file:
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@@
+    )
+  )
+  (symbol (lib_id "DPX165950DT-8126A1:DPX165950DT-8126A1") (at 179.705 233.045 0) (unit 1)
+    (in_bom yes) (on_board yes) (dnp no) (fields_autoplaced)
+    (property "Reference" "U5" (at 217.805 223.52 0)
+      (effects (font (size 1.524 1.524)))
+    )
+    (property "Value" "DPX165950DT-8126A1" (at 217.805 226.06 0)
+      (effects (font (size 1.524 1.524)))
+    )
+    (property "Footprint" "DPX165950DT-8126A1:DPX-6_1P6X0P8" (at 179.705 233.045 0)
+      (effects (font (size 1.27 1.27) italic) hide)
+    )
+    (property "Datasheet" "DPX165950DT-8126A1" (at 179.705 233.045 0)
+      (effects (font (size 1.27 1.27) italic) hide)
+    )
+    (pin "3")
+    (pin "4")
+    (pin "1")
+    (pin "6")
+    (pin "5")
+    (pin "2")
+    (instances
+      (project "DualWatch"
+        (path "/9c47ae17-f150-4290-a1ee-d756173e0f3d/a96f8989-b3b9-49ae-bafb-2cce3366f8fb"
+          (reference "U5") (unit 1)
+        )
+      )
     )
   )
@@
         )
       )
-    )
-  )
-  (symbol (lib_id "DPX165950DT-8126A1:DPX165950DT-8126A1") (at 179.705 233.045 0) (unit 1)
-    (in_bom yes) (on_board yes) (dnp no) (fields_autoplaced)
-    (property "Reference" "U5" (at 217.805 222.885 0)
-      (effects (font (size 1.524 1.524)))
-    )
-    (property "Value" "DPX165950DT-8126A1" (at 217.805 225.425 0)
-      (effects (font (size 1.524 1.524)))
-    )
-    (property "Footprint" "Package_LGA:LGA-16_3x3mm_P0.5mm_LayoutBorder3x5y" (at 179.705 233.045 0)
-      (effects (font (size 1.27 1.27) italic) hide)
-    )
-    (property "Datasheet" "DPX165950DT-8126A1" (at 179.705 233.045 0)
-      (effects (font (size 1.27 1.27) italic) hide)
-    )
-    (pin "4")
-    (pin "2")
-    (pin "1")
-    (pin "5")
-    (pin "3")
-    (pin "6")
-    (instances
-      (project "DualWatch"
-        (path "/9c47ae17-f150-4290-a1ee-d756173e0f3d/a96f8989-b3b9-49ae-bafb-2cce3366f8fb"
-          (reference "U5") (unit 1)
-        )
-      )

Commit message: update pcb placing
Parts:
- C30, C33, C36, C37, C39, C40, C42, C45, C46: footprint Capacitor_SMD:C_0603_1608Metric -> Capacitor_SMD:C_0402_1005Metric
Changed lines of the file:
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@@
       (effects (font (size 1.27 1.27)) (justify left))
     )
-    (property "Footprint" "Capacitor_SMD:C_0603_1608Metric" (at 211.7852 119.38 0)
+    (property "Footprint" "Capacitor_SMD:C_0402_1005Metric" (at 211.7852 119.38 0)
       (effects (font (size 1.27 1.27)) hide)
     )
@@
       (effects (font (size 1.27 1.27)) (justify left))
     )
-    (property "Footprint" "Capacitor_SMD:C_0603_1608Metric" (at 244.8052 115.57 0)
+    (property "Footprint" "Capacitor_SMD:C_0402_1005Metric" (at 244.8052 115.57 0)
       (effects (font (size 1.27 1.27)) hide)
     )
@@
       (effects (font (size 1.27 1.27)) (justify left))
     )
-    (property "Footprint" "Capacitor_SMD:C_0603_1608Metric" (at 280.3652 106.045 0)
+    (property "Footprint" "Capacitor_SMD:C_0402_1005Metric" (at 280.3652 106.045 0)
       (effects (font (size 1.27 1.27)) hide)
     )
@@
       (effects (font (size 1.27 1.27)) (justify left))
     )
-    (property "Footprint" "Capacitor_SMD:C_0603_1608Metric" (at 253.6952 119.38 0)
+    (property "Footprint" "Capacitor_SMD:C_0402_1005Metric" (at 253.6952 119.38 0)
       (effects (font (size 1.27 1.27)) hide)
     )
@@
       (effects (font (size 1.27 1.27)) (justify left))
     )
-    (property "Footprint" "Capacitor_SMD:C_0603_1608Metric" (at 263.2202 115.57 0)
+    (property "Footprint" "Capacitor_SMD:C_0402_1005Metric" (at 263.2202 115.57 0)
       (effects (font (size 1.27 1.27)) hide)
     )
@@
       (effects (font (size 1.27 1.27)) (justify left))
     )
-    (property "Footprint" "Capacitor_SMD:C_0603_1608Metric" (at 228.2952 58.42 0)
+    (property "Footprint" "Capacitor_SMD:C_0402_1005Metric" (at 228.2952 58.42 0)
       (effects (font (size 1.27 1.27)) hide)
     )
@@
       (effects (font (size 1.27 1.27)) (justify left))
     )
-    (property "Footprint" "Capacitor_SMD:C_0603_1608Metric" (at 305.1302 92.71 0)
+    (property "Footprint" "Capacitor_SMD:C_0402_1005Metric" (at 305.1302 92.71 0)
       (effects (font (size 1.27 1.27)) hide)
     )
@@
       (effects (font (size 1.27 1.27)) (justify left))
     )
-    (property "Footprint" "Capacitor_SMD:C_0603_1608Metric" (at 240.3602 59.055 0)
+    (property "Footprint" "Capacitor_SMD:C_0402_1005Metric" (at 240.3602 59.055 0)
       (effects (font (size 1.27 1.27)) hide)
     )
@@
       (effects (font (size 1.27 1.27)) (justify left))
     )
-    (property "Footprint" "Capacitor_SMD:C_0603_1608Metric" (at 314.6552 88.265 0)
-      (effects (font (size 1.27 1.27)) hide)
-    )
+    (property "Footprint" "Capacitor_SMD:C_0402_1005Metric" (at 314.6552 88.265 0)
+      (effects (font (size 1.27 1.27)) hide)
+    )
