File: Hardware/DualWatch/DualWatch.kicad_sch (KiCad schematic)
At the start: 0 parts

Commit message: Update Schematic
Other:
- added sheet DC DC (dc-regulators.kicad_sch)
- added sheet Peripheral (peripheral.kicad_sch)
- sheet nPM1100 ports: added VBAT; removed none
Changed lines of the file:
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@@
 (kicad_sch (version 20230121) (generator eeschema)
   (paper "A4")
+  (wire (pts (xy 65.405 56.515) (xy 65.405 72.39))
+    (stroke (width 0) (type default))
+  )
   (wire (pts (xy 100.33 53.34) (xy 104.775 53.34))
     (stroke (width 0) (type default))
@@
     (stroke (width 0) (type default))
   )
+  (wire (pts (xy 101.6 71.12) (xy 104.775 71.12))
+    (stroke (width 0) (type default))
+  )
   (wire (pts (xy 147.955 56.515) (xy 153.035 56.515))
     (stroke (width 0) (type default))
@@
     (stroke (width 0) (type default))
   )
+  (wire (pts (xy 101.6 89.535) (xy 104.775 89.535))
+    (stroke (width 0) (type default))
+  )
+  (wire (pts (xy 69.85 56.515) (xy 65.405 56.515))
+    (stroke (width 0) (type default))
+  )
   (wire (pts (xy 147.955 112.395) (xy 153.035 112.395))
     (stroke (width 0) (type default))
   )
+  (wire (pts (xy 101.6 84.455) (xy 104.775 84.455))
+    (stroke (width 0) (type default))
+  )
   (wire (pts (xy 100.33 57.15) (xy 104.775 57.15))
     (stroke (width 0) (type default))
@@
     (stroke (width 0) (type default))
   )
+  (wire (pts (xy 101.6 86.995) (xy 104.775 86.995))
+    (stroke (width 0) (type default))
+  )
+  (wire (pts (xy 101.6 81.915) (xy 104.775 81.915))
+    (stroke (width 0) (type default))
+  )
   (wire (pts (xy 147.955 120.015) (xy 153.035 120.015))
     (stroke (width 0) (type default))
@@
     (stroke (width 0) (type default))
   )
+  (wire (pts (xy 101.6 92.075) (xy 104.775 92.075))
+    (stroke (width 0) (type default))
+  )
   (wire (pts (xy 147.955 85.09) (xy 153.035 85.09))
     (stroke (width 0) (type default))
@@
     (stroke (width 0) (type default))
   )
+  (wire (pts (xy 101.6 73.66) (xy 104.775 73.66))
+    (stroke (width 0) (type default))
+  )
   (wire (pts (xy 100.33 59.055) (xy 104.775 59.055))
     (stroke (width 0) (type default))
@@
     (stroke (width 0) (type default))
   )
+  (wire (pts (xy 65.405 72.39) (xy 69.85 72.39))
+    (stroke (width 0) (type default))
+  )
   (wire (pts (xy 100.33 49.53) (xy 104.775 49.53))
     (stroke (width 0) (type default))
@@
       (effects (font (size 1.27 1.27)) (justify right))
     )
+    (pin "VBAT" input (at 69.85 56.515 180)
+      (effects (font (size 1.27 1.27)) (justify left))
+    )
     (instances
       (project "DualWatch"
@@
     )
   )
+  (sheet (at 69.85 69.215) (size 31.75 6.35) (fields_autoplaced)
+    (stroke (width 0.1524) (type solid))
+    (fill (color 0 0 0 0.0000))
+    (property "Sheetname" "DC DC" (at 69.85 68.5034 0)
+      (effects (font (size 1.27 1.27)) (justify left bottom))
+    )
+    (property "Sheetfile" "dc-regulators.kicad_sch" (at 69.85 76.1496 0)
+      (effects (font (size 1.27 1.27)) (justify left top))
+    )
+    (pin "WAKE_UP" input (at 101.6 71.12 0)
+      (effects (font (size 1.27 1.27)) (justify right))
+    )
+    (pin "VBAT" input (at 69.85 72.39 180)
+      (effects (font (size 1.27 1.27)) (justify left))
+    )
+    (pin "REG_ENABLE" input (at 101.6 73.66 0)
+      (effects (font (size 1.27 1.27)) (justify right))
+    )
+    (instances
+      (project "DualWatch"
+        (path "/9c47ae17-f150-4290-a1ee-d756173e0f3d" (page "7"))
+      )
+    )
+  )
   (sheet (at 153.035 83.185) (size 24.13 10.16) (fields_autoplaced)
     (stroke (width 0.1524) (type solid))
@@
       (effects (font (size 1.27 1.27)) (justify left))
     )
-    (pin "P0.05{slash}AIN1" input (at 104.775 76.835 180)
+    (pin "P0.05{slash}AIN1" input (at 104.775 84.455 180)
       (effects (font (size 1.27 1.27)) (justify left))
     )
@@
       (effects (font (size 1.27 1.27)) (justify right))
     )
-    (pin "P0.06{slash}AIN2" input (at 104.775 79.375 180)
-      (effects (font (size 1.27 1.27)) (justify left))
-    )
-    (pin "P0.07{slash}AIN3" input (at 104.775 81.915 180)
+    (pin "P0.06{slash}AIN2" input (at 104.775 86.995 180)
+      (effects (font (size 1.27 1.27)) (justify left))
+    )
+    (pin "P0.07{slash}AIN3" input (at 104.775 89.535 180)
       (effects (font (size 1.27 1.27)) (justify left))
     )
@@
       (effects (font (size 1.27 1.27)) (justify right))
     )
-    (pin "P1.12" input (at 104.775 71.755 180)
-      (effects (font (size 1.27 1.27)) (justify left))
-    )
-    (pin "P1.13" input (at 104.775 74.295 180)
+    (pin "P1.12" input (at 104.775 73.66 180)
+      (effects (font (size 1.27 1.27)) (justify left))
+    )
+    (pin "P1.13" input (at 104.775 81.915 180)
       (effects (font (size 1.27 1.27)) (justify left))
     )
@@
       (effects (font (size 1.27 1.27)) (justify left))
     )
-    (pin "P1.11" input (at 104.775 69.215 180)
+    (pin "P1.11" input (at 104.775 71.12 180)
       (effects (font (size 1.27 1.27)) (justify left))
     )
@@
       (effects (font (size 1.27 1.27)) (justify left))
     )
-    (pin "P0.25{slash}AIN4" input (at 104.775 89.535 180)
+    (pin "P0.25{slash}AIN4" input (at 104.775 97.155 180)
       (effects (font (size 1.27 1.27)) (justify left))
     )
@@
       (effects (font (size 1.27 1.27)) (justify right))
     )
-    (pin "P0.26{slash}AIN5" input (at 104.775 86.995 180)
-      (effects (font (size 1.27 1.27)) (justify left))
-    )
-    (pin "P0.27{slash}AIN6" input (at 104.775 84.455 180)
+    (pin "P0.26{slash}AIN5" input (at 104.775 94.615 180)
+      (effects (font (size 1.27 1.27)) (justify left))
+    )
+    (pin "P0.27{slash}AIN6" input (at 104.775 92.075 180)
       (effects (font (size 1.27 1.27)) (justify left))
     )
@@
       )
     )
+  )
+  (sheet (at 69.85 80.645) (size 31.75 19.685) (fields_autoplaced)
+    (stroke (width 0.1524) (type solid))
+    (fill (color 0 0 0 0.0000))
+    (property "Sheetname" "Peripheral" (at 69.85 79.9334 0)
+      (effects (font (size 1.27 1.27)) (justify left bottom))
+    )
+    (property "Sheetfile" "peripheral.kicad_sch" (at 69.85 100.9146 0)
+      (effects (font (size 1.27 1.27)) (justify left top))
+    )
+    (pin "LED-1" input (at 101.6 84.455 0)
+      (effects (font (size 1.27 1.27)) (justify right))
+    )
+    (pin "LED-2" input (at 101.6 86.995 0)
+      (effects (font (size 1.27 1.27)) (justify right))
+    )
+    (pin "LED-3" input (at 101.6 89.535 0)
+      (effects (font (size 1.27 1.27)) (justify right))
+    )
+    (pin "LED-4" input (at 101.6 92.075 0)
+      (effects (font (size 1.27 1.27)) (justify right))
+    )
+    (pin "BTN" input (at 101.6 81.915 0)
+      (effects (font (size 1.27 1.27)) (justify right))
+    )
+    (instances
+      (project "DualWatch"
+        (path "/9c47ae17-f150-4290-a1ee-d756173e0f3d" (page "8"))
+      )
+    )

Commit message: update pcb
Other:
- sheet WIFI ports: added VDDIO; removed IOVDD
Changed lines of the file:
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@@
       (effects (font (size 1.27 1.27)) (justify left))
     )
-    (pin "IOVDD" input (at 153.035 74.295 180)
+    (pin "VDDIO" input (at 153.035 74.295 180)
       (effects (font (size 1.27 1.27)) (justify left))
     )

Commit message: update pcb
Connections:
- no-connect marks 0 -> 1
Other:
- sheet MCU ports: added none; removed USB_D+, USB_D-
- sheet nPM1100 ports: added none; removed ISET, USB-D+, USB-D-
Changed lines of the file:
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@@
 (kicad_sch (version 20230121) (generator eeschema)
   (paper "A4")
+  (no_connect (at 104.775 47.625))
   (wire (pts (xy 65.405 56.515) (xy 65.405 72.39))
     (stroke (width 0) (type default))
@@
     (stroke (width 0) (type default))
   )
-  (wire (pts (xy 100.33 47.625) (xy 104.775 47.625))
-    (stroke (width 0) (type default))
-  )
   (wire (pts (xy 147.955 86.995) (xy 153.035 86.995))
     (stroke (width 0) (type default))
@@
     (stroke (width 0) (type default))
   )
-  (wire (pts (xy 100.33 45.72) (xy 104.775 45.72))
-    (stroke (width 0) (type default))
-  )
   (wire (pts (xy 147.955 90.805) (xy 153.035 90.805))
     (stroke (width 0) (type default))
@@
     (stroke (width 0) (type default))
   )
-  (wire (pts (xy 100.33 43.815) (xy 104.775 43.815))
-    (stroke (width 0) (type default))
-  )
   (wire (pts (xy 101.6 92.075) (xy 104.775 92.075))
     (stroke (width 0) (type default))
@@
     (stroke (width 0) (type default))
   )
-  (sheet (at 69.85 41.91) (size 30.48 19.05) (fields_autoplaced)
-    (stroke (width 0.1524) (type solid))
-    (fill (color 0 0 0 0.0000))
-    (property "Sheetname" "nPM1100" (at 69.85 41.1984 0)
+  (sheet (at 69.85 45.72) (size 30.48 15.24) (fields_autoplaced)
+    (stroke (width 0.1524) (type solid))
+    (fill (color 0 0 0 0.0000))
+    (property "Sheetname" "nPM1100" (at 69.85 45.0084 0)
       (effects (font (size 1.27 1.27)) (justify left bottom))
     )
@@
       (effects (font (size 1.27 1.27)) (justify left top))
     )
-    (pin "USB-D+" input (at 100.33 43.815 0)
-      (effects (font (size 1.27 1.27)) (justify right))
-    )
-    (pin "USB-D-" input (at 100.33 45.72 0)
-      (effects (font (size 1.27 1.27)) (justify right))
-    )
-    (pin "ISET" input (at 100.33 47.625 0)
-      (effects (font (size 1.27 1.27)) (justify right))
-    )
     (pin "CHG" input (at 100.33 49.53 0)
       (effects (font (size 1.27 1.27)) (justify right))
@@
       (effects (font (size 1.27 1.27)) (justify right))
     )
-    (pin "USB_D+" input (at 104.775 43.815 180)
-      (effects (font (size 1.27 1.27)) (justify left))
-    )
-    (pin "USB_D-" input (at 104.775 45.72 180)
-      (effects (font (size 1.27 1.27)) (justify left))
-    )
     (instances
       (project "DualWatch"
@@
     )
   )
-  (sheet (at 69.85 80.645) (size 31.75 19.685) (fields_autoplaced)
+  (sheet (at 69.85 80.645) (size 31.75 13.97) (fields_autoplaced)
     (stroke (width 0.1524) (type solid))
     (fill (color 0 0 0 0.0000))
@@
       (effects (font (size 1.27 1.27)) (justify left bottom))
     )
-    (property "Sheetfile" "peripheral.kicad_sch" (at 69.85 100.9146 0)
-      (effects (font (size 1.27 1.27)) (justify left top))
-    )
+    (property "Sheetfile" "peripheral.kicad_sch" (at 69.85 95.1996 0)
+      (effects (font (size 1.27 1.27)) (justify left top))
+    )
