File: Hardware/DualWatch/gc9a01.kicad_sch (KiCad schematic)
At the start: 24 parts, among them Q1 BSS123, U10 SN74LV1T34DCK, U11 SN74LV1T34DCK, U12 SN74LV1T34DCK, U13 SN74LV1T34DCK, U14 SN74LV1T34DCK, U15 SN74LV1T34DCK, U16 SN74LV1T34DCK, U17 SN74LV1T34DCK, U18 SN74LV1T34DCK, U8 SN74LV1T34DCK, U9 SN74LV1T34DCK

Commit message: Update Schematic
Parts:
- renumbered R11 to R10, R7 to R11, R8 to R4, R10 to R5, R4 to R6, R5 to R7, R6 to R8, U18 to U17, U17 to U18

Commit message: update pcb placing
Parts:
- removed U9: SN74LV1T34DCK, Package_TO_SOT_SMD:SOT-353_SC-70-5, symbol Logic_LevelTranslator:SN74LV1T34DCK
Changed lines of the file:
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@@
-    (stroke (width 0) (type default))
-  )
-  (wire (pts (xy 59.055 74.295) (xy 52.07 74.295))
     (stroke (width 0) (type default))
   )
@@
     (effects (font (size 1.27 1.27)) (justify right bottom))
   )
-  (label "MISO" (at 59.055 74.295 180) (fields_autoplaced)
-    (effects (font (size 1.27 1.27)) (justify right bottom))
-  )
   (label "INT" (at 135.255 102.235 180) (fields_autoplaced)
     (effects (font (size 1.27 1.27)) (justify right bottom))
@@
   )
   (hierarchical_label "SPI_SCK" (shape input) (at 36.83 102.235 180) (fields_autoplaced)
-    (effects (font (size 1.27 1.27)) (justify right))
-  )
-  (hierarchical_label "SPI_MISO" (shape input) (at 36.83 74.295 180) (fields_autoplaced)
     (effects (font (size 1.27 1.27)) (justify right))
   )
@@
         (path "/9c47ae17-f150-4290-a1ee-d756173e0f3d/cb744824-cbe5-4873-97e4-b99a3d465da5"
           (reference "#PWR058") (unit 1)
-        )
-      )
-    )
-  )
-  (symbol (lib_id "power:GND") (at 44.45 81.915 0) (unit 1)
-    (in_bom yes) (on_board yes) (dnp no) (fields_autoplaced)
-    (property "Reference" "#PWR056" (at 44.45 88.265 0)
-      (effects (font (size 1.27 1.27)) hide)
-    )
-    (property "Value" "GND" (at 44.45 86.36 0)
-      (effects (font (size 1.27 1.27)))
-    )
-    (property "Footprint" "" (at 44.45 81.915 0)
-      (effects (font (size 1.27 1.27)) hide)
-    )
-    (property "Datasheet" "" (at 44.45 81.915 0)
-      (effects (font (size 1.27 1.27)) hide)
-    )
-    (pin "1")
-    (instances
-      (project "DualWatch"
-        (path "/9c47ae17-f150-4290-a1ee-d756173e0f3d/cb744824-cbe5-4873-97e4-b99a3d465da5"
-          (reference "#PWR056") (unit 1)
         )
       )
@@
     )
   )
-  (symbol (lib_id "power:+3V3") (at 44.45 66.675 0) (unit 1)
-    (in_bom yes) (on_board yes) (dnp no) (fields_autoplaced)
-    (property "Reference" "#PWR055" (at 44.45 70.485 0)
-      (effects (font (size 1.27 1.27)) hide)
-    )
-    (property "Value" "+3V3" (at 44.45 61.595 0)
-      (effects (font (size 1.27 1.27)))
-    )
-    (property "Footprint" "" (at 44.45 66.675 0)
-      (effects (font (size 1.27 1.27)) hide)
-    )
-    (property "Datasheet" "" (at 44.45 66.675 0)
-      (effects (font (size 1.27 1.27)) hide)
-    )
-    (pin "1")
-    (instances
-      (project "DualWatch"
-        (path "/9c47ae17-f150-4290-a1ee-d756173e0f3d/cb744824-cbe5-4873-97e4-b99a3d465da5"
-          (reference "#PWR055") (unit 1)
-        )
-      )
-    )
-  )
   (symbol (lib_id "Device:R") (at 185.42 66.675 0) (unit 1)
     (in_bom yes) (on_board yes) (dnp no) (fields_autoplaced)
@@
         )
       )
-    )
-  )
-  (symbol (lib_id "Logic_LevelTranslator:SN74LV1T34DCK") (at 44.45 74.295 0) (unit 1)
-    (in_bom yes) (on_board yes) (dnp no)
-    (property "Reference" "U9" (at 55.245 64.135 0)
-      (effects (font (size 1.27 1.27)))
-    )
-    (property "Value" "SN74LV1T34DCK" (at 55.245 66.675 0)
-      (effects (font (size 1.27 1.27)))
-    )
-    (property "Footprint" "Package_TO_SOT_SMD:SOT-353_SC-70-5" (at 64.77 80.645 0)
-      (effects (font (size 1.27 1.27)) hide)
-    )
-    (property "Datasheet" "https://www.ti.com/lit/ds/symlink/sn74lv1t34.pdf" (at 34.29 79.375 0)
-      (effects (font (size 1.27 1.27)) hide)
-    )
-    (pin "3")
-    (pin "4")
-    (pin "5")
-    (pin "1")
-    (pin "2")
-    (instances
-      (project "DualWatch"
-        (path "/9c47ae17-f150-4290-a1ee-d756173e0f3d/cb744824-cbe5-4873-97e4-b99a3d465da5"
-          (reference "U9") (unit 1)
-        )
-      )

Commit message: update pcb
Parts:
- renumbered U11 to U10, U12 to U11, U13 to U12, U14 to U13, U15 to U14, U16 to U15, U17 to U16, U18 to U17, U19 to U18, U10 to U9
