File: Hardware/DualWatch/peripheral.kicad_sch (KiCad schematic)
At the start: 10 parts

Commit message: update pcb
Parts:
- renumbered R28 to R26, R29 to R27, R30 to R28, R31 to R29, R32 to R30
Changed lines of the file:
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@@
   (symbol (lib_id "Device:R") (at 62.865 69.215 90) (unit 1)
     (in_bom yes) (on_board yes) (dnp no) (fields_autoplaced)
-    (property "Reference" "R30" (at 62.865 62.865 90)
+    (property "Reference" "R28" (at 62.865 62.865 90)
       (effects (font (size 1.27 1.27)))
     )
@@
       (project "DualWatch"
         (path "/9c47ae17-f150-4290-a1ee-d756173e0f3d/fa838c20-6d60-46ca-8c20-8f7bef4ad30f"
-          (reference "R30") (unit 1)
+          (reference "R28") (unit 1)
         )
       )
@@
   (symbol (lib_id "Device:R") (at 66.04 114.935 0) (unit 1)
     (in_bom yes) (on_board yes) (dnp no) (fields_autoplaced)
-    (property "Reference" "R32" (at 67.945 113.665 0)
+    (property "Reference" "R30" (at 67.945 113.665 0)
       (effects (font (size 1.27 1.27)) (justify left))
     )
@@
       (project "DualWatch"
         (path "/9c47ae17-f150-4290-a1ee-d756173e0f3d/fa838c20-6d60-46ca-8c20-8f7bef4ad30f"
-          (reference "R32") (unit 1)
+          (reference "R30") (unit 1)
         )
       )
@@
   (symbol (lib_id "Device:R") (at 62.865 59.055 90) (unit 1)
     (in_bom yes) (on_board yes) (dnp no) (fields_autoplaced)
-    (property "Reference" "R29" (at 62.865 52.705 90)
+    (property "Reference" "R27" (at 62.865 52.705 90)
       (effects (font (size 1.27 1.27)))
     )
@@
       (project "DualWatch"
         (path "/9c47ae17-f150-4290-a1ee-d756173e0f3d/fa838c20-6d60-46ca-8c20-8f7bef4ad30f"
-          (reference "R29") (unit 1)
+          (reference "R27") (unit 1)
         )
       )
@@
   (symbol (lib_id "Device:R") (at 62.23 80.645 90) (unit 1)
     (in_bom yes) (on_board yes) (dnp no) (fields_autoplaced)
-    (property "Reference" "R28" (at 62.23 74.295 90)
+    (property "Reference" "R26" (at 62.23 74.295 90)
       (effects (font (size 1.27 1.27)))
     )
@@
       (project "DualWatch"
         (path "/9c47ae17-f150-4290-a1ee-d756173e0f3d/fa838c20-6d60-46ca-8c20-8f7bef4ad30f"
-          (reference "R28") (unit 1)
+          (reference "R26") (unit 1)
         )
       )
@@
   (symbol (lib_id "power:GND") (at 43.815 128.905 0) (unit 1)
     (in_bom yes) (on_board yes) (dnp no) (fields_autoplaced)
-    (property "Reference" "#PWR0115" (at 43.815 135.255 0)
+    (property "Reference" "#PWR0108" (at 43.815 135.255 0)
       (effects (font (size 1.27 1.27)) hide)
     )
@@
       (project "DualWatch"
         (path "/9c47ae17-f150-4290-a1ee-d756173e0f3d/fa838c20-6d60-46ca-8c20-8f7bef4ad30f"
-          (reference "#PWR0115") (unit 1)
+          (reference "#PWR0108") (unit 1)
         )
       )
@@
   (symbol (lib_id "power:GND") (at 72.39 85.725 0) (unit 1)
     (in_bom yes) (on_board yes) (dnp no) (fields_autoplaced)
-    (property "Reference" "#PWR0117" (at 72.39 92.075 0)
+    (property "Reference" "#PWR0110" (at 72.39 92.075 0)
       (effects (font (size 1.27 1.27)) hide)
     )
@@
       (project "DualWatch"
         (path "/9c47ae17-f150-4290-a1ee-d756173e0f3d/fa838c20-6d60-46ca-8c20-8f7bef4ad30f"
-          (reference "#PWR0117") (unit 1)
+          (reference "#PWR0110") (unit 1)
         )
       )
@@
   (symbol (lib_id "Device:R") (at 63.5 48.26 90) (unit 1)
     (in_bom yes) (on_board yes) (dnp no) (fields_autoplaced)
-    (property "Reference" "R31" (at 63.5 41.91 90)
+    (property "Reference" "R29" (at 63.5 41.91 90)
       (effects (font (size 1.27 1.27)))
     )
@@
       (project "DualWatch"
         (path "/9c47ae17-f150-4290-a1ee-d756173e0f3d/fa838c20-6d60-46ca-8c20-8f7bef4ad30f"
-          (reference "R31") (unit 1)
+          (reference "R29") (unit 1)
         )
       )
@@
   (symbol (lib_id "power:+1V8") (at 66.04 109.22 0) (unit 1)
     (in_bom yes) (on_board yes) (dnp no) (fields_autoplaced)
-    (property "Reference" "#PWR0116" (at 66.04 113.03 0)
+    (property "Reference" "#PWR0109" (at 66.04 113.03 0)
       (effects (font (size 1.27 1.27)) hide)
     )
@@
       (project "DualWatch"
         (path "/9c47ae17-f150-4290-a1ee-d756173e0f3d/fa838c20-6d60-46ca-8c20-8f7bef4ad30f"
-          (reference "#PWR0116") (unit 1)
-        )
-      )
+          (reference "#PWR0109") (unit 1)
+        )
+      )
