File: Hardware/DualWatch/DualWatch.kicad_pcb (KiCad board)
At the start: 4 copper layers, 0 parts

Commit message: Update pcb
Parts:
- added C1: 30nF, Capacitor_SMD:C_0402_1005Metric, F.Cu at (158.1, 125.3)
- added C10: 1uF, Capacitor_SMD:C_0402_1005Metric, F.Cu at (158.1, 133.2)
- added C11: 2.2nF, Capacitor_SMD:C_0603_1608Metric, F.Cu at (171.3, 125.6)
- added C12: 2.2uF, Capacitor_SMD:C_0402_1005Metric, F.Cu at (158.1, 135.2)
- added C13: 4.7uF, Capacitor_SMD:C_0603_1608Metric, F.Cu at (171.3, 128.1)
- added C14: 100nF, Capacitor_SMD:C_0603_1608Metric, F.Cu at (171.3, 130.6)
- added C15: 1uF, Capacitor_SMD:C_0402_1005Metric, F.Cu at (158.1, 137.1)
- added C16: 1uF, Capacitor_SMD:C_0402_1005Metric, F.Cu at (161.0, 125.3)
- added C17: 100nF, Capacitor_SMD:C_0603_1608Metric, F.Cu at (171.3, 133.1)
- added C18: 100nF, Capacitor_SMD:C_0402_1005Metric, F.Cu at (161.0, 127.3)
- added C19: 1uF, Capacitor_SMD:C_0402_1005Metric, F.Cu at (161.0, 129.2)
- added C2: 30nF, Capacitor_SMD:C_0402_1005Metric, F.Cu at (158.1, 127.3)
- added C20: 100nF, Capacitor_SMD:C_0402_1005Metric, F.Cu at (161.0, 131.2)
- added C21: 100nF, Capacitor_SMD:C_0402_1005Metric, F.Cu at (161.0, 133.2)
- added C22: 0.7pF, Capacitor_SMD:C_0402_1005Metric, F.Cu at (161.0, 135.2)
- added C23: 100nF, Capacitor_SMD:C_0402_1005Metric, F.Cu at (161.0, 137.1)
- added C24: 100nF, Capacitor_SMD:C_0402_1005Metric, F.Cu at (163.9, 125.3)
- added C25: NC, Capacitor_SMD:C_0402_1005Metric, F.Cu at (163.9, 127.3)
- added C26: 100nF, Capacitor_SMD:C_0603_1608Metric, F.Cu at (171.3, 135.6)
- added C27: 100nF, Capacitor_SMD:C_0402_1005Metric, F.Cu at (163.9, 129.2)
- added C28: 1uF, Capacitor_SMD:C_0402_1005Metric, F.Cu at (163.9, 131.2)
- added C29: 100nF, Capacitor_SMD:C_0402_1005Metric, F.Cu at (186.7, 83.7)
- added C3: 30nF, Capacitor_SMD:C_0402_1005Metric, F.Cu at (158.1, 129.2)
- added C30: 10nF, Capacitor_SMD:C_0603_1608Metric, F.Cu at (178.9, 96.4)
- added C31: 100nF, Capacitor_SMD:C_0402_1005Metric, F.Cu at (183.4, 85.2)
- added C32: 4.7uF, Capacitor_SMD:C_0603_1608Metric, F.Cu at (176.7, 98.7)
- added C33: 470nF, Capacitor_SMD:C_0603_1608Metric, F.Cu at (177.5, 83.8)
- added C34: 1uF, Capacitor_SMD:C_0402_1005Metric, F.Cu at (183.3, 95.8)
- added C35: 2.2uF, Capacitor_SMD:C_0402_1005Metric, F.Cu at (184.3, 95.8)
- added C36: 100nF, Capacitor_SMD:C_0603_1608Metric, F.Cu at (173.6, 83.1)
- added C37: 470nF, Capacitor_SMD:C_0603_1608Metric, F.Cu at (182.0, 96.4)
- added C38: 4.7uF, Capacitor_SMD:C_0603_1608Metric, F.Cu at (175.9, 83.8)
- added C39: 2.2uF, Capacitor_SMD:C_0603_1608Metric, F.Cu at (184.7, 85.8)
- added C4: 30nF, Capacitor_SMD:C_0402_1005Metric, F.Cu at (158.1, 131.2)
- added C40: 2.2uF, Capacitor_SMD:C_0603_1608Metric, F.Cu at (180.5, 96.4)
- added C41: 4.7uF, Capacitor_SMD:C_0603_1608Metric, F.Cu at (175.9, 96.4)
- added C42: 1uF, Capacitor_SMD:C_0603_1608Metric, F.Cu at (173.6, 95.6)
- added C43: 1uF, Capacitor_SMD:C_0402_1005Metric, F.Cu at (174.1, 94.3)
- added C44: 2.2uF, Capacitor_SMD:C_0402_1005Metric, F.Cu at (174.1, 89.0)
- added C45: 220nF, Capacitor_SMD:C_0603_1608Metric, F.Cu at (173.6, 87.7)
- added C46: 22nF, Capacitor_SMD:C_0603_1608Metric, F.Cu at (173.6, 86.2)
- added C47: 4.7uF, Capacitor_SMD:C_0603_1608Metric, F.Cu at (173.6, 84.6)
- added C48: 100nF, Capacitor_SMD:C_0603_1608Metric, F.Cu at (21.2, 99.0)
- added C49: 10uF, Capacitor_SMD:C_0603_1608Metric, F.Cu at (21.2, 101.5)
- added C5: 4.7uF, Capacitor_SMD:C_0603_1608Metric, F.Cu at (167.3, 125.6)
- added C50: 100nF, Capacitor_SMD:C_0603_1608Metric, F.Cu at (21.2, 104.0)
- added C51: 10uF, Capacitor_SMD:C_0603_1608Metric, F.Cu at (66.7, 48.7)
- added C52: 1uF, Capacitor_SMD:C_0603_1608Metric, F.Cu at (66.7, 51.3)
- added C53: 10uF, Capacitor_SMD:C_0603_1608Metric, F.Cu at (66.7, 53.8)
- added C54: 10uF, Capacitor_SMD:C_0603_1608Metric, F.Cu at (66.7, 56.3)
- added C55: 2.2uF, Capacitor_SMD:C_0603_1608Metric, F.Cu at (66.7, 58.8)
- added C56: 10uF, Capacitor_SMD:C_0603_1608Metric, F.Cu at (51.4, 55.3)
- added C57: 100nF, Capacitor_SMD:C_0402_1005Metric, F.Cu at (60.6, 63.2)
- added C58: 10uF, Capacitor_SMD:C_0603_1608Metric, F.Cu at (51.4, 57.9)
- added C59: 100nF, Capacitor_SMD:C_0402_1005Metric, F.Cu at (60.6, 65.1)
- added C6: 1uF, Capacitor_SMD:C_0603_1608Metric, F.Cu at (167.3, 128.1)
- added C60: 10uF, Capacitor_SMD:C_0402_1005Metric, F.Cu at (60.6, 67.1)
- added C61: 10uF, Capacitor_SMD:C_0402_1005Metric, F.Cu at (60.6, 69.1)
- added C62: 10uF, Capacitor_SMD:C_0603_1608Metric, F.Cu at (51.4, 60.4)
- added C63: 10uF, Capacitor_SMD:C_0603_1608Metric, F.Cu at (51.4, 62.9)
- added C7: 1uF, Capacitor_SMD:C_0603_1608Metric, F.Cu at (167.3, 130.6)
- added C8: 4.7uF, Capacitor_SMD:C_0603_1608Metric, F.Cu at (167.3, 133.1)
- added C9: 1uF, Capacitor_SMD:C_0603_1608Metric, F.Cu at (167.3, 135.6)
- added D1: LED, LED_SMD:LED_0603_1608Metric, F.Cu at (80.0, 56.6)
- added D2: LED, LED_SMD:LED_0603_1608Metric, F.Cu at (80.0, 59.2)
- added D3: MBR0520, Diode_SMD:D_SOD-123, F.Cu at (56.3, 63.9)
- added D4: MBR0520, Diode_SMD:D_SOD-123, F.Cu at (56.3, 67.2)
- added D5: LED, LED_SMD:LED_0603_1608Metric, F.Cu at (66.8, 65.8)
- added D6: LED, LED_SMD:LED_0603_1608Metric, F.Cu at (66.8, 68.4)
- added D7: LED, LED_SMD:LED_0603_1608Metric, F.Cu at (66.8, 71.0)
- added D8: LED, LED_SMD:LED_0603_1608Metric, F.Cu at (66.8, 73.6)
- added F1: 6V/1.5A, Fuse:Fuse_0805_2012Metric, F.Cu at (148.2, 103.4)
- added J1: NFC, Connector_PinHeader_1.27mm:PinHeader_1x02_P1.27mm_Vertical, F.Cu at (158.8, 148.2)
- added J2: NRF_Debug, Connector_PinHeader_1.27mm:PinHeader_2x05_P1.27mm_Vertical, F.Cu at (158.8, 139.8)
- added J3: USB_C_Receptacle_USB2.0, Connector_USB:USB_C_Receptacle_HRO_TYPE-C-31-M-12, F.Cu at (144.6, 109.7)
- added J4: Conn_01x02_Pin, Connector_PinHeader_2.54mm:PinHeader_1x02_P2.54mm_Vertical, F.Cu at (79.6, 49.8)
- added L1: 10uH, Inductor_SMD:L_0603_1608Metric, F.Cu at (179.6, 125.7)
- added L10: 8.7nH, Inductor_SMD:L_0603_1608Metric, F.Cu at (179.3, 78.1)
- added L11: 8.2nH, Inductor_SMD:L_0402_1005Metric, F.Cu at (178.8, 76.0)
- added L12: 6.8nH, Inductor_SMD:L_0603_1608Metric, F.Cu at (179.3, 73.9)
- added L13: 2.2uH, Inductor_SMD:L_6.3x6.3_H3, F.Cu at (73.0, 51.4)
- added L14: 1.5uH, Inductor_SMD:L_Coilcraft_XAL4020-XXX, F.Cu at (46.4, 50.5)
- added L15: 1.5uH, Inductor_SMD:L_Coilcraft_XAL4020-XXX, F.Cu at (46.4, 56.4)
- added L2: 10uH, Inductor_SMD:L_0603_1608Metric, F.Cu at (179.6, 128.4)
- added L3: 10uH, Inductor_SMD:L_0603_1608Metric, F.Cu at (179.6, 131.2)
- added L4: 10uH, Inductor_SMD:L_0603_1608Metric, F.Cu at (175.3, 125.6)
- added L5: 8.7nH, Inductor_SMD:L_0603_1608Metric, F.Cu at (175.3, 128.1)
- added L6: 8.2nH, Inductor_SMD:L_0402_1005Metric, F.Cu at (163.6, 139.1)
- added L7: 6.8nH, Inductor_SMD:L_0603_1608Metric, F.Cu at (175.3, 130.6)
- added L8: 220R, Inductor_SMD:L_0603_1608Metric, F.Cu at (179.6, 133.9)
- added L9: 3.3uH, Inductor_SMD:L_0603_1608Metric, F.Cu at (177.4, 96.4)
- added Q1: BSS123, Package_TO_SOT_SMD:SOT-23, F.Cu at (39.0, 49.7)
- added Q2: IRLM2803, Package_TO_SOT_SMD:SOT-23, F.Cu at (60.3, 49.7)
- added R1: 2.2R, Resistor_SMD:R_0402_1005Metric, F.Cu at (163.6, 141.1)
- added R10: 10K, Resistor_SMD:R_0402_1005Metric, F.Cu at (39.0, 57.4)
- added R11: 10K, Resistor_SMD:R_0402_1005Metric, F.Cu at (39.0, 59.4)
- added R12: 1K, Resistor_SMD:R_0402_1005Metric, F.Cu at (39.0, 61.4)
- added R13: 10K, Resistor_SMD:R_0402_1005Metric, F.Cu at (39.0, 63.4)
- added R14: 10R, Resistor_SMD:R_0402_1005Metric, F.Cu at (39.0, 65.4)
- added R15: 1M5, Resistor_SMD:R_0402_1005Metric, F.Cu at (76.5, 56.3)
- added R16: 220K, Resistor_SMD:R_0402_1005Metric, F.Cu at (76.5, 58.3)
- added R17: 1.5K, Resistor_SMD:R_0402_1005Metric, F.Cu at (76.5, 60.3)
- added R18: 100K, Resistor_SMD:R_0402_1005Metric, F.Cu at (44.9, 60.4)
- added R19: 100K, Resistor_SMD:R_0402_1005Metric, F.Cu at (44.9, 62.4)
- added R2: 5.1K, Resistor_SMD:R_0402_1005Metric, F.Cu at (143.3, 103.4)
- added R20: 200K, Resistor_SMD:R_0402_1005Metric, F.Cu at (44.9, 64.3)
- added R21: 100K, Resistor_SMD:R_0402_1005Metric, F.Cu at (44.9, 66.3)
- added R22: 178K, Resistor_SMD:R_0402_1005Metric, F.Cu at (44.9, 68.3)
- added R23: 261K, Resistor_SMD:R_0402_1005Metric, F.Cu at (47.8, 60.4)
- added R24: 1M, Resistor_SMD:R_0402_1005Metric, F.Cu at (47.8, 62.4)
- added R25: 1K, Resistor_SMD:R_0402_1005Metric, F.Cu at (47.8, 64.3)
- added R26: 10K, Resistor_SMD:R_0402_1005Metric, F.Cu at (47.8, 66.3)
- added R27: 10K, Resistor_SMD:R_0402_1005Metric, F.Cu at (47.8, 68.3)
- added R28: 100R, Resistor_SMD:R_0402_1005Metric, F.Cu at (70.2, 65.5)
- added R29: 100R, Resistor_SMD:R_0402_1005Metric, F.Cu at (70.2, 67.5)
- added R3: 5.1K, Resistor_SMD:R_0402_1005Metric, F.Cu at (146.0, 103.4)
- added R30: 100R, Resistor_SMD:R_0402_1005Metric, F.Cu at (70.2, 69.5)
- added R31: 100R, Resistor_SMD:R_0402_1005Metric, F.Cu at (70.2, 71.5)
- added R32: 10K, Resistor_SMD:R_0402_1005Metric, F.Cu at (70.2, 73.5)
- added R4: 10K, Resistor_SMD:R_0402_1005Metric, F.Cu at (36.1, 57.4)
- added R5: 10K, Resistor_SMD:R_0402_1005Metric, F.Cu at (36.1, 59.4)
- added R6: 10K, Resistor_SMD:R_0402_1005Metric, F.Cu at (36.1, 61.4)
- added R7: 10K, Resistor_SMD:R_0402_1005Metric, F.Cu at (36.1, 63.4)
- added R8: 10K, Resistor_SMD:R_0402_1005Metric, F.Cu at (36.1, 65.4)
- added R9: 10K, Resistor_SMD:R_0402_1005Metric, F.Cu at (36.1, 67.4)
- added SW1: ~, EVQ-PSD02K:EVQ-PSD02K, F.Cu at (53.0, 50.8)
- added SW2: ~, EVQ-PSD02K:EVQ-PSD02K, F.Cu at (75.3, 67.8)
- added TH1: 10K, Resistor_SMD:R_0603_1608Metric, F.Cu at (66.7, 61.3)
- added U1: NRF5340-QKAA-R7, Footprints:XCVR_NRF5340-QKAA-R7, F.Cu at (181.8, 141.1)
- added U10: SN74LV1T34DCK, Package_TO_SOT_SMD:SOT-353_SC-70-5, F.Cu at (24.0, 66.1)
- added U11: SN74LV1T34DCK, Package_TO_SOT_SMD:SOT-353_SC-70-5, F.Cu at (24.0, 69.9)
- added U12: SN74LV1T34DCK, Package_TO_SOT_SMD:SOT-353_SC-70-5, F.Cu at (28.2, 58.4)
- added U13: SN74LV1T34DCK, Package_TO_SOT_SMD:SOT-353_SC-70-5, F.Cu at (28.2, 62.2)
- added U14: SN74LV1T34DCK, Package_TO_SOT_SMD:SOT-353_SC-70-5, F.Cu at (28.2, 66.1)
- added U15: SN74LV1T34DCK, Package_TO_SOT_SMD:SOT-353_SC-70-5, F.Cu at (28.2, 69.9)
- added U16: SN74LV1T34DCK, Package_TO_SOT_SMD:SOT-353_SC-70-5, F.Cu at (32.5, 58.4)
- added U17: SN74LV1T34DCK, Package_TO_SOT_SMD:SOT-353_SC-70-5, F.Cu at (32.5, 62.2)
- added U18: SN74LV1T34DCK, Package_TO_SOT_SMD:SOT-353_SC-70-5, F.Cu at (32.5, 66.1)
- added U19: ~, 1-28-LCD-Touch:1.28LCD-TP, F.Cu at (18.2, 50.0)
- added U2: ~, nn02-101:NN02-101, F.Cu at (179.5, 148.4)
- added U20: NPM1100-QDAA-R7, NPM1100-QDAA-R7:QFN24_NPM1100_NOR, F.Cu at (71.9, 58.6)
- added U21: TPS63030DSK, Package_SON:WSON-10-1EP_2.5x2.5mm_P0.5mm_EP1.2x2mm, F.Cu at (55.8, 56.1)
- added U22: TPS63030DSK, Package_SON:WSON-10-1EP_2.5x2.5mm_P0.5mm_EP1.2x2mm, F.Cu at (55.8, 60.2)
- added U23: SN74LV1T34DCK, Package_TO_SOT_SMD:SOT-353_SC-70-5, F.Cu at (60.3, 56.0)
- added U24: SN74LV1T34DCK, Package_TO_SOT_SMD:SOT-353_SC-70-5, F.Cu at (60.3, 59.9)
- added U3: 74LVC1G3157, Package_TO_SOT_SMD:SOT-23-6, F.Cu at (187.2, 86.4)
- added U4: NRF7002-QFAA-R, Footprints:IC_NRF7002-QFAA-R, F.Cu at (180.2, 90.1)
- added U5: DPX165950DT-8126A1, DPX165950DT-8126A1:DPX-6_1P6X0P8, F.Cu at (179.4, 81.0)
- added U6: ~, nn02-101:NN02-101, F.Cu at (178.3, 69.8)
- added U7: LIS3DH, Package_LGA:LGA-16_3x3mm_P0.5mm_LayoutBorder3x5y, F.Cu at (25.5, 100.0)
- added U8: SN74LV1T34DCK, Package_TO_SOT_SMD:SOT-353_SC-70-5, F.Cu at (24.0, 58.4)
- added U9: SN74LV1T34DCK, Package_TO_SOT_SMD:SOT-353_SC-70-5, F.Cu at (24.0, 62.2)
- added Y1: 32.768kHz, Crystal:Crystal_SMD_3215-2Pin_3.2x1.5mm, F.Cu at (173.1, 149.0)
- added Y2: 32MHz, Crystal:Crystal_SMD_3225-4Pin_3.2x2.5mm, F.Cu at (167.9, 149.6)
- added Y3: 40Mhz, Crystal:Crystal_SMD_3225-4Pin_3.2x2.5mm, F.Cu at (173.3, 91.6)
Other:
- board outline added: 41.2 x 42.1 mm

Commit message: update pcb placing
Parts:
- removed U9: SN74LV1T34DCK, Package_TO_SOT_SMD:SOT-353_SC-70-5
- C11, C14, C17, C26, C30, C33, C36, C37, C39, C40, C42, C45, C46, C48, C50, C52, C55, C6, C7, C9: footprint Capacitor_SMD:C_0603_1608Metric -> Capacitor_SMD:C_0402_1005Metric
- C56, C57, C58, C59, C62, C63, L14, L15, R21, R22, R23, R24, R28, R29, R30, R31, U10, U11, U12, U13, U14, U15, U16, U17, U18, U19, U21, U22, U8: moved to B.Cu
- C60, C61: footprint Capacitor_SMD:C_0402_1005Metric -> Capacitor_SMD:C_0603_1608Metric; moved to B.Cu
- L1, L12, L2, L3, L8: footprint Inductor_SMD:L_0603_1608Metric -> Inductor_SMD:L_0805_2012Metric
- L13: footprint Inductor_SMD:L_6.3x6.3_H3 -> Inductor_SMD:L_Coilcraft_XAL4020-XXX
- moved L14 176.4 mm to (202.3, 133.0)
- moved C56 173.7 mm to (204.6, 137.1), turned to -90 degrees
- moved R21 171.2 mm to (200.1, 138.5), turned to 90 degrees
- moved R23 170.4 mm to (200.2, 136.6), turned to 90 degrees
- moved L15 169.6 mm to (205.1, 116.1)
- moved C58 168.1 mm to (207.4, 120.2), turned to -90 degrees
- moved U21 167.6 mm to (202.2, 137.5), turned to -90 degrees
- moved R22 166.8 mm to (203.0, 121.5), turned to 90 degrees
- moved C62 166.3 mm to (198.9, 137.1), turned to -90 degrees
- moved R24 165.4 mm to (203.0, 119.5), turned to 90 degrees
- moved C57 161.1 mm to (202.2, 140.0)
- moved U22 161.1 mm to (205.1, 120.6), turned to -90 degrees
- moved C63 159.8 mm to (201.7, 117.0), turned to 90 degrees
- moved C59 155.6 mm to (205.1, 123.0)
- moved C60 153.7 mm to (198.9, 134.1), turned to 90 degrees
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Connections:
- U1 pad AK2: /LCD/SPI_MISO -> /MCU/P0.10/MISO

Commit message: update pcb
Parts:
- D3, D4, Q1, Q2, R10, R11, R12, R13, R14, R18, R19, R20, R27, R4, R5, R6, R7, R8, R9, U23, U24: moved to B.Cu
- moved R14 67.9 mm to (136.8, 80.1), turned to -90 degrees
- moved R13 65.7 mm to (137.8, 80.1), turned to 90 degrees
- moved R8 65.7 mm to (150.8, 79.9), turned to 90 degrees
- moved C56 65.5 mm to (149.7, 101.4)
- moved R23 65.5 mm to (145.2, 100.9)
- moved C62 65.5 mm to (143.9, 101.4)
- moved L14 65.5 mm to (147.4, 97.3)
- moved C57 65.5 mm to (147.3, 104.3)
- moved C60 65.5 mm to (144.0, 98.4)
- moved R21 65.5 mm to (145.2, 102.8)
- moved U21 65.5 mm to (147.3, 101.8)
- moved R9 65.2 mm to (144.5, 82.8)
- moved R12 64.4 mm to (135.6, 80.1), turned to -90 degrees
- moved R7 63.7 mm to (152.8, 79.9), turned to 90 degrees
- moved R10 63.3 mm to (144.7, 75.2)
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Connections:
- U3 pad 6: /WIFI/VDDIO -> /MCU/P0.31
Routing:
- net /MCU/USB_D-: track 0.00 -> 58.5 mm, vias 0 -> 2
- net /MCU/USB_D+: track 0.00 -> 56.2 mm
- net +1V8: track 0.00 -> 29.9 mm, vias 0 -> 11
- net +3V3: track 0.00 -> 16.0 mm, vias 0 -> 2
- net Net-(U1A-DECR): track 0.00 -> 10.3 mm, vias 0 -> 2
- net /MCU/XL1: track 0.00 -> 9.02 mm, vias 0 -> 2
- net /nPM1100/VSYS: track 0.00 -> 8.88 mm
- net /DC DC/VBAT: track 0.00 -> 8.24 mm, vias 0 -> 1
- net Net-(D4-A): track 0.00 -> 7.84 mm
- net /MCU/P1.13: track 0.00 -> 7.48 mm
- net /MCU/XC2: track 0.00 -> 7.09 mm
- net /WIFI/XOP: track 0.00 -> 6.67 mm
- net Net-(U1A-DCCH): track 0.00 -> 6.16 mm, vias 0 -> 2
- net Net-(U1A-DCCD): track 0.00 -> 6.13 mm, vias 0 -> 2
- net /MCU/XC1: track 0.00 -> 6.11 mm
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- added copper zone on In2.Cu, net +1V8
- added copper zone on In1.Cu, net +3V3
- added copper zone on B.Cu, net GND
- added copper zone on F.Cu, net GND

Commit message: update pcb
Parts:
- removed C60, C61, C62, C63: 10uF, Capacitor_SMD:C_0603_1608Metric
- removed L15: 1.5uH, Inductor_SMD:L_Coilcraft_XAL4020-XXX
- removed R31: 100R, Resistor_SMD:R_0402_1005Metric
- removed R32: 10K, Resistor_SMD:R_0402_1005Metric
- removed U23, U24: SN74LV1T34DCK, Package_TO_SOT_SMD:SOT-353_SC-70-5
- added U9: SN74LV1T34DCK, Package_TO_SOT_SMD:SOT-353_SC-70-5, B.Cu at (139.2, 90.4)
- C59: value 100nF -> 10uF; footprint Capacitor_SMD:C_0402_1005Metric -> Capacitor_SMD:C_0603_1608Metric
- D4, Q2, R18: moved to F.Cu
- L8: moved to B.Cu
- R21: value 100K -> 178K
- R22: value 178K -> 1M
- R23: value 261K -> 1K; moved to F.Cu
- R24: value 1M -> 10K; moved to F.Cu
- R25: value 1K -> 10K
- R26: value 10K -> 100R; moved to B.Cu
- R27: value 10K -> 100R
- R30: value 100R -> 10K; moved to F.Cu
- U18: value SN74LV1T34DCK -> ~; footprint Package_TO_SOT_SMD:SOT-353_SC-70-5 -> 1-28-LCD-Touch:1.28LCD-TP
- U19: value ~ -> NPM1100-QDAA-R7; footprint 1-28-LCD-Touch:1.28LCD-TP -> NPM1100-QDAA-R7:QFN24_NPM1100_NOR; moved to F.Cu
- U20: value NPM1100-QDAA-R7 -> TPS63030DSK; footprint NPM1100-QDAA-R7:QFN24_NPM1100_NOR -> Package_SON:WSON-10-1EP_2.5x2.5mm_P0.5mm_EP1.2x2mm; moved to B.Cu
- U21, U22: value TPS63030DSK -> SN74LV1T34DCK; footprint Package_SON:WSON-10-1EP_2.5x2.5mm_P0.5mm_EP1.2x2mm -> Package_TO_SOT_SMD:SOT-353_SC-70-5; moved to F.Cu
- moved R30 40.5 mm to (122.0, 89.3), turned to 60 degrees
- moved C58 36.1 mm to (121.4, 97.7)
- moved C59 34.9 mm to (121.4, 94.6), turned to 90 degrees
- moved U22 33.6 mm to (122.2, 94.1), turned to 180 degrees
- moved U20 32.7 mm to (124.7, 101.4), turned to -90 degrees
- moved J4 32.2 mm to (157.6, 95.4), turned to 180 degrees
- moved R15 32.1 mm to (158.1, 97.8), turned to 0 degrees
- moved R16 32.1 mm to (158.1, 98.8), turned to 180 degrees
- moved R22 30.3 mm to (122.7, 100.4)
- moved R19 27.5 mm to (125.8, 104.3), turned to 90 degrees
- moved D5 27.3 mm to (136.6, 105.1), turned to 90 degrees
- moved J2 27.2 mm to (148.3, 112.5), turned to 135 degrees
- moved R20 27.0 mm to (126.8, 104.3), turned to -90 degrees
- moved R29 26.4 mm to (136.6, 105.4), turned to 90 degrees
- moved U21 25.5 mm to (122.3, 97.0), turned to 180 degrees
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Connections:
- C54 pad 2: Net-(U20-DEC) -> Net-(U19-DEC)
- C57 pad 2: Net-(U21-PS/SYNC) -> Net-(U20-PS/SYNC)
- C58 pad 1: VIN -> +3V3
- C59 pad 1: GND -> +3V3
- C59 pad 2: Net-(U22-PS/SYNC) -> GND
- L13 pad 1: Net-(U20-SW) -> Net-(U19-SW)
- L14 pad 1: Net-(U21-L2) -> Net-(U20-L2)
- L14 pad 2: Net-(U21-L1) -> Net-(U20-L1)
- R17 pad 1: Net-(U20-ICHG) -> Net-(U19-ICHG)
- R21 pad 2: Net-(U21-FB) -> Net-(U20-FB)
- R22 pad 1: GND -> Net-(U20-FB)
- R22 pad 2: Net-(U22-FB) -> +3V3
- R23 pad 1: Net-(U21-FB) -> /DC DC/BTN
- R23 pad 2: +1V8 -> Net-(D4-A)
- R24 pad 1: Net-(U22-FB) -> Net-(D4-A)
- R24 pad 2: +3V3 -> GND
- R25 pad 1: /DC DC/BTN -> /DC DC/REG_EN
- R25 pad 2: Net-(D4-A) -> GND
- R26 pad 1: Net-(D4-A) -> Net-(D8-K)
- R27 pad 1: /DC DC/REG_EN -> Net-(D6-K)
- R28 pad 1: Net-(D8-K) -> Net-(D7-K)
- R29 pad 1: Net-(D6-K) -> Net-(D5-K)
- R30 pad 1: Net-(D7-K) -> +1V8
- R30 pad 2: GND -> /MCU/P1.13
- TH1 pad 1: Net-(U20-NTC) -> Net-(U19-NTC)
- U10 pad 2: /LCD/SPI_SCK -> /LCD/SPI_CS
- U10 pad 4: /LCD/SCK -> /LCD/CS
- U11 pad 2: /LCD/SPI_CS -> /LCD/LCD_DC
- U11 pad 4: /LCD/CS -> /LCD/DC
- U12 pad 2: /LCD/LCD_DC -> /LCD/LCD_RESET
- U12 pad 4: /LCD/DC -> /LCD/LCD_RST
- U13 pad 2: /LCD/LCD_RESET -> /LCD/LCD_BL
- U13 pad 4: /LCD/LCD_RST -> /LCD/BL
- U14 pad 2: /LCD/LCD_BL -> /LCD/I2C_SDA
- U14 pad 4: /LCD/BL -> /LCD/SDA
- U15 pad 2: /LCD/I2C_SDA -> /LCD/I2C_SCL
- U15 pad 4: /LCD/SDA -> /LCD/SCL
- U16 pad 2: /LCD/I2C_SCL -> /LCD/TP_RESET
- U16 pad 4: /LCD/SCL -> /LCD/TP_RST
- U17 pad 2: /LCD/TP_RESET -> /LCD/TP_INT
- U17 pad 4: /LCD/TP_RST -> /LCD/INT
- U18 pad 1: unconnected-(U18-NC-Pad1) -> GND
- U18 pad 2: /LCD/TP_INT -> /LCD/LEDK
- U18 pad 3: GND -> +3V3
- U18 pad 4: /LCD/INT -> +3V3
- U18 pad 5: +3V3 -> /LCD/DC
- U19 pad 1: GND -> +1V8
- U19 pad 10: +3V3 -> /MCU/P1.07
- U19 pad 11: GND -> /MCU/P1.09
- U19 pad 12: /LCD/TP_RST -> Net-(U19-ICHG)
- U19 pad 13: /LCD/INT -> unconnected-(U19-NC-Pad13)
- U19 pad 14: /LCD/SDA -> Net-(U19-NTC)
- U19 pad 15: /LCD/SCL -> /DC DC/VBAT
- U19 pad 2: /LCD/LEDK -> GND
- U19 pad 3: +3V3 -> GND
- U19 pad 4: +3V3 -> unconnected-(U19-NC-Pad4)
- U19 pad 5: /LCD/DC -> /nPM1100/VSYS
- U19 pad 6: /LCD/CS -> /MCU/P1.10
- U19 pad 7: /LCD/SCK -> /MCU/P1.08
- U19 pad 8: /LCD/MOSI -> /MCU/P1.06
- U19 pad 9: /LCD/LCD_RST -> /nPM1100/VSYS
- U20 pad 1: +1V8 -> +3V3
- U20 pad 10: /MCU/P1.07 -> Net-(U20-FB)
- U20 pad 11: /MCU/P1.09 -> GND
- U20 pad 2: GND -> Net-(U20-L2)
- U20 pad 4: unconnected-(U20-NC-Pad4) -> Net-(U20-L1)
- U20 pad 5: /MCU/P1.05 -> VIN
- U20 pad 6: /MCU/P1.10 -> /DC DC/REG_EN
- U20 pad 7: /MCU/P1.08 -> Net-(U20-PS/SYNC)
- U20 pad 8: /MCU/P1.06 -> Net-(U20-PS/SYNC)
- U20 pad 9: /nPM1100/VSYS -> GND
- U21 pad 1: +1V8 -> unconnected-(U21-NC-Pad1)
- U21 pad 2: Net-(U21-L2) -> /DC DC/REG_ENABLE
- U21 pad 4: Net-(U21-L1) -> /DC DC/REG_EN
- U21 pad 5: VIN -> +3V3
- U22 pad 1: +3V3 -> unconnected-(U22-NC-Pad1)
- U22 pad 2: Net-(U22-L2) -> /DC DC/BTN
- U22 pad 4: Net-(U22-L1) -> /DC DC/WAKE_UP
- U22 pad 5: VIN -> +1V8
Routing:
- net /MCU/USB_D-: track 58.5 -> 0.00 mm, vias 2 -> 0
- net /MCU/USB_D+: track 56.2 -> 0.00 mm
- net +1V8: track 29.9 -> 0.00 mm, vias 11 -> 0
- net +3V3: track 16.0 -> 0.00 mm, vias 2 -> 0
- net Net-(U1A-DECR): track 10.3 -> 0.00 mm, vias 2 -> 0
- net /MCU/XL1: track 9.02 -> 0.00 mm, vias 2 -> 0
- net /nPM1100/VSYS: track 8.88 -> 0.00 mm
- net /DC DC/VBAT: track 8.24 -> 0.00 mm, vias 1 -> 0
- net Net-(D4-A): track 7.84 -> 0.00 mm
- net /MCU/P1.13: track 7.48 -> 0.00 mm
- net /MCU/XC2: track 7.09 -> 0.00 mm
- net /WIFI/XOP: track 6.67 -> 0.00 mm
- net Net-(U1A-DCCH): track 6.16 -> 0.00 mm, vias 2 -> 0
- net Net-(U1A-DCCD): track 6.13 -> 0.00 mm, vias 2 -> 0
- net /MCU/XC1: track 6.11 -> 0.00 mm
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- removed copper zone on In2.Cu, net +1V8
- removed copper zone on B.Cu, net GND
- removed copper zone on F.Cu, net GND
Other:
- board size 41.2 x 42.1 mm -> 40 x 41 mm

Commit message: update pcb
Parts:
- moved C57 2.86 mm to (124.8, 104.2), turned to 90 degrees
- moved C15 1.01 mm to (126.7, 101.5)
- moved C6 1.00 mm to (126.7, 102.5)
Routing:
- net +3V3: track 0.00 -> 185.6 mm, vias 0 -> 14
- net VBUS: track 0.00 -> 90.4 mm, vias 0 -> 6
- net /DC DC/BTN: track 0.00 -> 55.2 mm, vias 0 -> 2
- net +1V8: track 0.00 -> 53.3 mm, vias 0 -> 23
- net VIN: track 0.00 -> 52.0 mm, vias 0 -> 2
- net /DC DC/REG_EN: track 0.00 -> 50.6 mm, vias 0 -> 2
- net /DC DC/VBAT: track 0.00 -> 49.8 mm, vias 0 -> 4
- net /MCU/SWDCLK: track 0.00 -> 42.6 mm, vias 0 -> 2
- net /MCU/SWDIO: track 0.00 -> 39.3 mm, vias 0 -> 1
- net /MCU/P0.04/AIN0: track 0.00 -> 35.2 mm, vias 0 -> 2
- net /MCU/P1.10: track 0.00 -> 32.0 mm, vias 0 -> 3
- net /MCU/P0.30: track 0.00 -> 32.0 mm, vias 0 -> 3
- net /LCD/I2C_SDA: track 0.00 -> 31.6 mm, vias 0 -> 2
- net /MCU/NRESET: track 0.00 -> 31.3 mm, vias 0 -> 1
- net /MCU/P0.31: track 0.00 -> 30.0 mm, vias 0 -> 2
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- added copper zone on In2.Cu, net +1V8
- added copper zone on F.Cu, net +3V3
- added copper zone on B.Cu, net /DC DC/REG_EN
- added copper zone on B.Cu, net GND
- added copper zone on F.Cu, net GND
- added copper zone on In1.Cu, net GND
- added copper zone on B.Cu, net Net-(U20-L1)
- added copper zone on B.Cu, net Net-(U20-L2)
- added copper zone on B.Cu, net Net-(U20-PS/SYNC)
- removed copper zone on In1.Cu, net +3V3

Commit message: Finish Board
Parts:
- L14: footprint Inductor_SMD:L_Coilcraft_XAL4020-XXX -> Inductor_SMD:L_Murata_DFE201610P
- moved L14 1.40 mm to (124.7, 98.1)
Routing:
- net GND: track 14.5 -> 29.3 mm, vias 10 -> 16
- net /nPM1100/VSYS: track 18.7 -> 32.2 mm
- net VIN: track 52.0 -> 62.5 mm
- net Net-(D5-K): track 0.00 -> 1.17 mm, vias 0 -> 1
- net Net-(D6-K): track 0.00 -> 1.15 mm, vias 0 -> 1
- net Net-(D8-K): track 0.00 -> 1.13 mm, vias 0 -> 1
- net Net-(D7-K): track 0.00 -> 0.89 mm, vias 0 -> 1
- net /DC DC/REG_ENABLE: track 9.01 -> 9.88 mm
- net /MCU/P0.31: track 30.0 -> 30.8 mm
- net /WIFI/SW_CTRL0: track 0.81 -> 0.00 mm, vias 1 -> 0
- net /MCU/P1.05: vias 1 -> 0
- net /MCU/P0.25/AIN4: vias 1 -> 0
- net /MCU/P0.10/MISO: vias 1 -> 0

Commit message: Update pcb
Routing:
- net /MCU/NRESET: track 31.3 -> 32.4 mm
- net /WIFI/PWRIOVDD: track 17.8 -> 18.7 mm
- net VIN: track 62.5 -> 63.2 mm
- net /MCU/P0.27/AIN6: track 17.3 -> 18.0 mm
- net /MCU/SWDIO: track 39.3 -> 39.9 mm
- net /MCU/SWDCLK: track 42.6 -> 43.2 mm

Commit message: Update pcb
Parts:
- added kibuzzard-666B077B: G***, kibuzzard-666B077B, F.Cu at (129.2, 82.2)
- added kibuzzard-666B078A: G***, kibuzzard-666B078A, F.Cu at (151.8, 82.2)
- added kibuzzard-666B084B: G***, kibuzzard-666B084B, F.Cu at (156.8, 90.0)
- added kibuzzard-666B0874: G***, kibuzzard-666B0874, F.Cu at (123.8, 90.6)
- added kibuzzard-666B0889: G***, kibuzzard-666B0889, B.Cu at (153.4, 95.4)
- added kibuzzard-666B0895: G***, kibuzzard-666B0895, B.Cu at (153.2, 92.8)
Routing:
- net GND: vias 16 -> 110
